File: hardware/distance-ir-v2.kicad_pcb (KiCad board)
At the start: 2 copper layers, 18.9 x 44.6 mm, 23 parts, among them P1 CON-SENSOR2, P2 DEBUG, P3 BOOT, P4 S3B-PH-SM4, U2 DRILL, U3 DRILL, U4 XMC1XXX24

Commit message: improve routing, add distance led
Parts:
- removed R1: DNP, kicad-libraries:R0603F
- added D2: green, kicad-libraries:D0603E, F.Cu at (149.7, 112.6)
- added Fiducial_Mark: VAL**, kicad-libraries:Fiducial_Mark, F.Cu at (149.4, 104.8)
- added R4: 1k, kicad-libraries:R0603F, F.Cu at (139.3, 94.1)
- moved Fiducial_Mark 7.02 mm to (140.9, 115.3)
- moved P2 0.96 mm to (138.9, 90.9)
- moved R2 0.78 mm to (141.4, 97.1), turned to 90 degrees
Connections:
- U4 pad 11: Net-(U4-Pad11) -> (no net)
- U4 pad 12: Net-(U4-Pad12) -> (no net)
- U4 pad 13: Net-(U4-Pad13) -> Net-(P2-Pad1)
- U4 pad 15: Net-(P2-Pad1) -> (no net)
- U4 pad 16: Net-(U4-Pad16) -> (no net)
- U4 pad 17: Net-(U4-Pad17) -> (no net)
- U4 pad 18: Net-(U4-Pad18) -> (no net)
- U4 pad 19: Net-(U4-Pad19) -> (no net)
- U4 pad 20: Net-(U4-Pad20) -> (no net)
- U4 pad 21: Net-(U4-Pad21) -> (no net)
- U4 pad 3: Net-(U4-Pad3) -> (no net)
- U4 pad 5: Net-(U4-Pad5) -> (no net)
- U4 pad 6: Net-(U4-Pad6) -> (no net)
- U4 pad 8: Net-(U4-Pad8) -> (no net)
Routing:
- net Net-(D2-Pad2): track 0.00 -> 31.5 mm
- net VCC: track 34.8 -> 46.0 mm
- net Net-(R4-Pad1): track 0.00 -> 3.29 mm
- net IN_1: track 9.57 -> 8.40 mm
- net GND: track 31.2 -> 30.5 mm, vias 16 -> 15
- net Net-(P4-Pad3): track 9.52 -> 8.98 mm
Other:
- board text added: "Distance"

Commit message: fix origin
Parts:
- moved C4 0.08 mm to (144.4, 103.9)
- moved G*** 0.08 mm to (144.1, 102.0)
- moved P3 0.08 mm to (147.1, 91.4)
- moved P4 0.08 mm to (132.1, 102.0)
- moved RP1 0.08 mm to (144.1, 96.7)
- moved C3 0.08 mm to (145.9, 96.6)
- moved D1 0.08 mm to (149.8, 91.4)
- moved D2 0.08 mm to (149.8, 112.6)
- moved R3 0.08 mm to (146.6, 88.7)
- moved R4 0.08 mm to (139.4, 94.1)
- moved VAL 0.08 mm to (144.1, 109.0)
- moved C1 0.08 mm to (143.1, 88.7)
- moved C2 0.08 mm to (142.0, 108.3)
- moved C5 0.08 mm to (142.9, 103.9)
- moved P1 0.08 mm to (151.0, 102.0)
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Other:
- outline, holes or cut-outs redrawn

Commit message: specify processor
Parts:
- U4: value XMC1XXX24 -> XMC13XX24
Changed lines of the file:
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@@
-(kicad_pcb (version 4) (host pcbnew 4.0.2+dfsg1-stable)
+(kicad_pcb (version 4) (host pcbnew 4.0.7-e2-6376~61~ubuntu18.04.1)
   (general
     (links 42)
     (no_connects 0)
-    (area 131.0325 79.484499 281.446922 163.016883)
+    (area 131.1825 79.509499 281.34691 163.416933)
     (thickness 1.6002)
     (drawings 27)
@@
       (effects (font (size 0.3 0.3) (thickness 0.075)))
     )
-    (fp_text value XMC1XXX24 (at 0 0.8 180) (layer F.Fab)
+    (fp_text value XMC13XX24 (at 0 0.8 180) (layer F.Fab)
       (effects (font (size 0.3 0.3) (thickness 0.075)))
     )
