File: hardware/distance-ir-v2.kicad_pcb (KiCad board)
At the start: 2 copper layers, 18.9 x 44.6 mm, 25 parts, among them P1 CON-SENSOR2, P2 DEBUG, P3 BOOT, P4 S3B-PH-SM4, U2 DRILL, U3 DRILL, U4 XMC13XX24

Commit message: specify processor
Parts:
- U4: value XMC13XX24 -> XMC1302
Changed lines of the file:
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@@
       (effects (font (size 0.3 0.3) (thickness 0.075)))
     )
-    (fp_text value XMC13XX24 (at 0 0.8 180) (layer F.Fab)
+    (fp_text value XMC1302 (at 0 0.8 180) (layer F.Fab)
       (effects (font (size 0.3 0.3) (thickness 0.075)))
     )
